Commit message: FEAT: add RealSense D435 RGBD camera sensor to URDF

File: urdf/crane_x7.gazebo.xacro (robot description, xacro)
@@ -115,3 +115,120 @@
     </gazebo>
   </xacro:macro>
+  <!-- Gazebo RGBD Camera Sensor -->
+  <xacro:macro name="gazebo_camera_sensor" params="parent_link">
+    <!-- Camera link -->
+    <link name="camera_link">
+      <inertial>
+        <mass value="0.01"/>
+        <origin xyz="0 0 0" rpy="0 0 0"/>
+        <inertia ixx="0.0001" ixy="0" ixz="0" iyy="0.0001" iyz="0" izz="0.0001"/>
+      </inertial>
+      <visual>
+        <origin xyz="0 0 0" rpy="0 0 0"/>
+        <geometry>
+          <box size="0.025 0.09 0.025"/>
+        </geometry>
+        <material name="camera_material">
+          <color rgba="0.1 0.1 0.1 1"/>
+        </material>
+      </visual>
+      <!-- Collision disabled to avoid self-collision with gripper in MoveIt -->
+      <!--
+      <collision>
+        <origin xyz="0 0 0" rpy="0 0 0"/>
+        <geometry>
+          <box size="0.025 0.09 0.025"/>
+        </geometry>
+      </collision>
+      -->
+    </link>
+    <!-- Camera joint -->
+    <joint name="camera_joint" type="fixed">
+      <parent link="${parent_link}"/>
+      <child link="camera_link"/>
+      <origin xyz="0.0 0.032 0.0191" rpy="-1.5708 -1.5708 0"/>
+    </joint>
+    <!-- Camera optical frame -->
+    <link name="camera_color_optical_frame"/>
+    <joint name="camera_color_optical_joint" type="fixed">
+      <parent link="camera_link"/>
+      <child link="camera_color_optical_frame"/>
+      <origin xyz="0 0 0" rpy="-1.5708 0 -1.5708"/>
+    </joint>
+    <link name="camera_depth_optical_frame"/>
+    <joint name="camera_depth_optical_joint" type="fixed">
+      <parent link="camera_link"/>
+      <child link="camera_depth_optical_frame"/>
+      <origin xyz="0 0 0" rpy="-1.5708 0 -1.5708"/>
+    </joint>
+    <!-- Gazebo Fortress RGB Camera -->
+    <gazebo reference="camera_link">
+      <sensor name="camera_color" type="camera">
+        <pose>0 0 0 0 0 0</pose>
+        <always_on>true</always_on>
+        <update_rate>30</update_rate>
+        <visualize>true</visualize>
+        <topic>camera/color</topic>
+        <enable_metrics>false</enable_metrics>
+        <camera name="camera_color">
+          <horizontal_fov>1.211</horizontal_fov>
+          <image>
+            <width>640</width>
+            <height>480</height>
+            <format>R8G8B8</format>
+          </image>
+          <clip>
+            <near>0.1</near>
+            <far>100</far>
+          </clip>
+          <noise>
+            <type>gaussian</type>
+            <mean>0.0</mean>
+            <stddev>0.007</stddev>
+          </noise>
+          <lens>
+            <intrinsics>
+              <fx>277.0</fx>
+              <fy>277.0</fy>
+              <cx>320.0</cx>
+              <cy>240.0</cy>
+              <s>0.0</s>
+            </intrinsics>
+          </lens>
+        </camera>
+      </sensor>
+    </gazebo>
+    <!-- Gazebo Fortress Depth Camera -->
+    <gazebo reference="camera_link">
+      <sensor name="camera_depth" type="depth_camera">
+        <pose>0 0 0 0 0 0</pose>
+        <always_on>true</always_on>
+        <update_rate>30</update_rate>
+        <visualize>true</visualize>
+        <topic>camera/depth</topic>
+        <enable_metrics>false</enable_metrics>
+        <camera name="camera_depth">
+          <horizontal_fov>1.211</horizontal_fov>
+          <image>
+            <width>640</width>
+            <height>480</height>
+            <format>R_FLOAT32</format>
+          </image>
+          <clip>
+            <near>0.1</near>
+            <far>10.0</far>
+          </clip>
+          <lens>
+            <intrinsics>
+              <fx>277.0</fx>
+              <fy>277.0</fy>
+              <cx>320.0</cx>
+              <cy>240.0</cy>
+              <s>0.0</s>
+            </intrinsics>
+          </lens>
+        </camera>
+      </sensor>
+    </gazebo>
+  </xacro:macro>
 </robot>

File: urdf/crane_x7.urdf.xacro (robot description, xacro)
@@ -258,4 +258,6 @@
       joint_hand_lower_limit="${JOINT_HAND_LOWER_LIMIT}"
       joint_hand_upper_limit="${JOINT_HAND_UPPER_LIMIT}" />
+    <!-- Add camera sensor for Gazebo -->
+    <xacro:gazebo_camera_sensor parent_link="${NAME_LINK_7}" />
   </xacro:if>
 </robot>

Commit message: FEAT: update URDF and description loader for improved accuracy

File: urdf/crane_x7.gazebo.xacro (robot description, xacro)
@@ -144,8 +144,11 @@
     </link>
     <!-- Camera joint -->
+    <!-- Camera mounted on gripper, pointing forward/down for hand-eye configuration -->
+    <!-- Offset: Y=0.032 (side), Z=0.0191 (up from gripper base) -->
+    <!-- Orientation: Looking along gripper's approach direction (downward when gripper is down) -->
     <joint name="camera_joint" type="fixed">
       <parent link="${parent_link}"/>
       <child link="camera_link"/>
-      <origin xyz="0.0 0.032 0.0191" rpy="-1.5708 -1.5708 0"/>
+      <origin xyz="0.0 0.032 0.0191" rpy="0 -1.5708 -1.5708"/>
     </joint>
     <!-- Camera optical frame -->
@@ -171,4 +174,5 @@
         <topic>camera/color</topic>
         <enable_metrics>false</enable_metrics>
+        <gz_frame_id>camera_color_optical_frame</gz_frame_id>
         <camera name="camera_color">
           <horizontal_fov>1.211</horizontal_fov>
@@ -208,4 +212,5 @@
         <topic>camera/depth</topic>
         <enable_metrics>false</enable_metrics>
+        <gz_frame_id>camera_depth_optical_frame</gz_frame_id>
         <camera name="camera_depth">
           <horizontal_fov>1.211</horizontal_fov>

File: urdf/crane_x7.xacro (robot description, xacro)
@@ -171,4 +171,5 @@
           add_plug="false"
           use_mesh="true">
+        <!-- Default mounting offset for crane_x7 D435 bracket -->
         <origin xyz="0.0 0.032 0.0191" rpy="${radians(-90)} ${radians(-90)} 0"/>
       </xacro:sensor_d435>
